Commit message: femur - fr bl

File: src/spiderbot_description/urdf/_back_right_leg.xacro (robot description, xacro)
@@ -18,3 +18,20 @@
         <limit lower="-${PI/2}" upper="${PI/4}" effort="${effort}" velocity="${velocity}" />
     </joint>
+    <link name="br_femur">
+        <visual>
+            <origin rpy="0 0 0" xyz="0.08 -0.23 0.0" />
+            <geometry>
+                <mesh filename="package://spiderbot_description/meshes/m_femur_flbr.stl"
+                    scale="0.01 0.01 0.01" />
+            </geometry>
+            <material name="green" />
+        </visual>
+    </link>
+    <joint name="joint_hip_femur_br" type="revolute">
+        <parent link="br_hip" />
+        <child link="br_femur" />
+        <origin rpy="0 0 ${-PI/2}" xyz="-0.33 0.0 0.03" />
+        <axis xyz="1 0 0"/>
+        <limit lower="-${PI/2}" upper="${PI/4}" effort="${effort}" velocity="${velocity}" />
+    </joint>
 </robot>

File: src/spiderbot_description/urdf/_front_left_leg.xacro (robot description, xacro)
@@ -18,3 +18,20 @@
         <limit lower="-${PI/2}" upper="${PI/4}" effort="${effort}" velocity="${velocity}" />
     </joint>
+    <link name="fl_femur">
+        <visual>
+            <origin rpy="0 0 0" xyz="0.08 -0.23 0.0" />
+            <geometry>
+                <mesh filename="package://spiderbot_description/meshes/m_femur_flbr.stl"
+                    scale="0.01 0.01 0.01" />
+            </geometry>
+            <material name="green" />
+        </visual>
+    </link>
+    <joint name="joint_hip_femur_fl" type="revolute">
+        <parent link="fl_hip" />
+        <child link="fl_femur" />
+        <origin rpy="0 0 ${PI/2}" xyz="0.33 0.0 0.03" />
+        <axis xyz="1 0 0"/>
+        <limit lower="-${PI/2}" upper="${PI/4}" effort="${effort}" velocity="${velocity}" />
+    </joint>
 </robot>

Commit message: All legs completed

File: src/spiderbot_description/urdf/_back_right_leg.xacro (robot description, xacro)
@@ -35,3 +35,20 @@
         <limit lower="-${PI/4}" upper="${PI/2}" effort="${effort}" velocity="${velocity}" />
     </joint>
+    <link name="br_tibia">
+        <visual>
+            <origin rpy="${PI} ${PI} ${PI}" xyz="0.01 0.26 0.0" />
+            <geometry>
+                <mesh filename="package://spiderbot_description/meshes/m_tibia_flbr.stl"
+                    scale="0.01 0.01 0.01" />
+            </geometry>
+            <material name="pink" />
+        </visual>
+    </link>
+    <joint name="joint_femur_tibia_br" type="revolute">
+        <parent link="br_femur" />
+        <child link="br_tibia" />
+        <origin rpy="0 0 0" xyz="0.0 0.46 0" />
+        <axis xyz="1 0 0"/>
+        <limit lower="-${4*PI/5}" upper="0" effort="${effort}" velocity="${velocity}" />
+    </joint>
 </robot>

File: src/spiderbot_description/urdf/_front_right_leg.xacro (robot description, xacro)
@@ -35,3 +35,20 @@
         <limit lower="-${PI/4}" upper="${PI/2}" effort="${effort}" velocity="${velocity}" />
     </joint>
+    <link name="fr_tibia">
+        <visual>
+            <origin rpy="${PI} ${PI} ${PI}" xyz="0.01 0.26 0.0" />
+            <geometry>
+                <mesh filename="package://spiderbot_description/meshes/m_tibia_frbl.stl"
+                    scale="0.01 0.01 0.01" />
+            </geometry>
+            <material name="purple" />
+        </visual>
+    </link>
+    <joint name="joint_femur_tibia_fr" type="revolute">
+        <parent link="fr_femur" />
+        <child link="fr_tibia" />
+        <origin rpy="0 0 0" xyz="0.0 0.46 0" />
+        <axis xyz="1 0 0"/>
+        <limit lower="-${4*PI/5}" upper="0" effort="${effort}" velocity="${velocity}" />
+    </joint>
 </robot>
