Commit message: All femurs

File: src/spiderbot_description/urdf/_back_left_leg.xacro (robot description, xacro)
@@ -18,3 +18,20 @@
         <limit lower="-${PI/4}" upper="${PI/2}" effort="${effort}" velocity="${velocity}" />
     </joint>
+    <link name="bl_femur">
+        <visual>
+            <origin rpy="${PI} ${PI} 0" xyz="0.08 0.23 0.0" />
+            <geometry>
+                <mesh filename="package://spiderbot_description/meshes/m_femur_frbl.stl"
+                    scale="0.01 0.01 0.01" />
+            </geometry>
+            <material name="yellow" />
+        </visual>
+    </link>
+    <joint name="joint_hip_femur_bl" type="revolute">
+        <parent link="bl_hip" />
+        <child link="bl_femur" />
+        <origin rpy="0 0 ${PI/2}" xyz="-0.33 0.0 0.03" />
+        <axis xyz="1 0 0"/>
+        <limit lower="-${PI/4}" upper="${PI/2}" effort="${effort}" velocity="${velocity}" />
+    </joint>
 </robot>

File: src/spiderbot_description/urdf/_front_right_leg.xacro (robot description, xacro)
@@ -18,3 +18,20 @@
         <limit lower="-${PI/4}" upper="${PI/2}" effort="${effort}" velocity="${velocity}" />
     </joint>
+    <link name="fr_femur">
+        <visual>
+            <origin rpy="${PI} ${PI} 0" xyz="0.08 0.23 0.0" />
+            <geometry>
+                <mesh filename="package://spiderbot_description/meshes/m_femur_frbl.stl"
+                    scale="0.01 0.01 0.01" />
+            </geometry>
+            <material name="yellow" />
+        </visual>
+    </link>
+    <joint name="joint_hip_femur_fr" type="revolute">
+        <parent link="fr_hip" />
+        <child link="fr_femur" />
+        <origin rpy="0 0 ${-PI/2}" xyz="0.33 0.0 0.03" />
+        <axis xyz="1 0 0"/>
+        <limit lower="-${PI/4}" upper="${PI/2}" effort="${effort}" velocity="${velocity}" />
+    </joint>
 </robot>

Commit message: BL rotated

File: src/spiderbot_description/urdf/_back_left_leg.xacro (robot description, xacro)
@@ -3,5 +3,5 @@
     <link name="bl_hip">
         <visual>
-            <origin rpy="0 0 0" xyz="-0.05 0 0" />
+            <origin rpy="${PI} 0 0" xyz="-0.05 0 0" />
             <geometry>
                 <mesh filename="package://spiderbot_description/meshes/m_coxa_frbl.stl"
@@ -14,11 +14,11 @@
         <parent link="base_link" />
         <child link="bl_hip" />
-        <origin rpy="0 0 0" xyz="-0.4 -0.37 0.06" />
+        <origin rpy="${PI} 0 0" xyz="-0.4 -0.37 0.06" />
         <axis xyz="0 0 1"/>
-        <limit lower="-${PI/4}" upper="${PI/2}" effort="${effort}" velocity="${velocity}" />
+        <limit lower="-${PI/2}" upper="${PI/4}" effort="${effort}" velocity="${velocity}" />
     </joint>
     <link name="bl_femur">
         <visual>
-            <origin rpy="${PI} ${PI} 0" xyz="0.08 0.23 0.0" />
+            <origin rpy="${PI} 0 ${PI}" xyz="0.08 -0.23 0.0" />
             <geometry>
                 <mesh filename="package://spiderbot_description/meshes/m_femur_frbl.stl"
@@ -31,7 +31,7 @@
         <parent link="bl_hip" />
         <child link="bl_femur" />
-        <origin rpy="0 0 ${PI/2}" xyz="-0.33 0.0 0.03" />
+        <origin rpy="0 0 ${-PI/2}" xyz="-0.33 0.0 0.03" />
         <axis xyz="1 0 0"/>
-        <limit lower="-${PI/4}" upper="${PI/2}" effort="${effort}" velocity="${velocity}" />
+        <limit lower="-${PI/2}" upper="${PI/4}" effort="${effort}" velocity="${velocity}" />
     </joint>
 </robot>

Commit message: Back legs rotated and aligned

File: src/spiderbot_description/urdf/_back_left_leg.xacro (robot description, xacro)
@@ -33,5 +33,5 @@
         <origin rpy="0 0 ${-PI/2}" xyz="-0.33 0.0 0.03" />
         <axis xyz="1 0 0"/>
-        <limit lower="-${PI/2}" upper="${PI/4}" effort="${effort}" velocity="${velocity}" />
+        <limit lower="-${PI/4}" upper="${PI/2}" effort="${effort}" velocity="${velocity}" />
     </joint>
 </robot>

File: src/spiderbot_description/urdf/_back_right_leg.xacro (robot description, xacro)
@@ -20,5 +20,5 @@
     <link name="br_femur">
         <visual>
-            <origin rpy="0 0 0" xyz="0.08 -0.23 0.0" />
+            <origin rpy="0 0 ${PI}" xyz="-0.08 0.23 0.0" />
             <geometry>
                 <mesh filename="package://spiderbot_description/meshes/m_femur_flbr.stl"
@@ -31,7 +31,7 @@
         <parent link="br_hip" />
         <child link="br_femur" />
-        <origin rpy="0 0 ${-PI/2}" xyz="-0.33 0.0 0.03" />
+        <origin rpy="0 0 ${PI/2}" xyz="-0.33 0.0 0.03" />
         <axis xyz="1 0 0"/>
-        <limit lower="-${PI/2}" upper="${PI/4}" effort="${effort}" velocity="${velocity}" />
+        <limit lower="-${PI/4}" upper="${PI/2}" effort="${effort}" velocity="${velocity}" />
     </joint>
 </robot>

Commit message: All legs moving in the same direction

File: src/spiderbot_description/urdf/_back_left_leg.xacro (robot description, xacro)
@@ -31,5 +31,5 @@
         <parent link="bl_hip" />
         <child link="bl_femur" />
-        <origin rpy="0 0 ${-PI/2}" xyz="-0.33 0.0 0.03" />
+        <origin rpy="0 0 ${-PI/2}" xyz="-0.33 0.0 -0.03" />
         <axis xyz="1 0 0"/>
         <limit lower="-${PI/4}" upper="${PI/2}" effort="${effort}" velocity="${velocity}" />

File: src/spiderbot_description/urdf/_front_left_leg.xacro (robot description, xacro)
@@ -3,5 +3,5 @@
     <link name="fl_hip">
         <visual>
-            <origin rpy="0 0 0" xyz="0.05 0 0" />
+            <origin rpy="${PI} 0 ${PI}" xyz="-0.05 0 0" />
             <geometry>
                 <mesh filename="package://spiderbot_description/meshes/m_coxa_flbr.stl"
@@ -14,11 +14,11 @@
         <parent link="base_link" />
         <child link="fl_hip" />
-        <origin rpy="0 0 ${PI}" xyz="-0.4 0.37 0.06" />
+        <origin rpy="${PI} 0 0" xyz="-0.4 0.37 0.06" />
         <axis xyz="0 0 1"/>
-        <limit lower="-${PI/2}" upper="${PI/4}" effort="${effort}" velocity="${velocity}" />
+        <limit lower="-${PI/4}" upper="${PI/2}" effort="${effort}" velocity="${velocity}" />
     </joint>
     <link name="fl_femur">
         <visual>
-            <origin rpy="0 0 0" xyz="0.08 -0.23 0.0" />
+            <origin rpy="${PI} 0 ${PI}" xyz="-0.08 -0.23 0.0" />
             <geometry>
                 <mesh filename="package://spiderbot_description/meshes/m_femur_flbr.stl"
@@ -31,7 +31,7 @@
         <parent link="fl_hip" />
         <child link="fl_femur" />
-        <origin rpy="0 0 ${PI/2}" xyz="0.33 0.0 0.03" />
+        <origin rpy="0 0 ${-PI/2}" xyz="-0.33 0.0 -0.03" />
         <axis xyz="1 0 0"/>
-        <limit lower="-${PI/2}" upper="${PI/4}" effort="${effort}" velocity="${velocity}" />
+        <limit lower="-${PI/4}" upper="${PI/2}" effort="${effort}" velocity="${velocity}" />
     </joint>
 </robot>

Commit message: Left feet

File: src/spiderbot_description/urdf/_back_left_leg.xacro (robot description, xacro)
@@ -35,3 +35,20 @@
         <limit lower="-${PI/4}" upper="${PI/2}" effort="${effort}" velocity="${velocity}" />
     </joint>
+    <link name="bl_tibia">
+        <visual>
+            <origin rpy="${PI} 0 0" xyz="0.01 -0.26 0.0" />
+            <geometry>
+                <mesh filename="package://spiderbot_description/meshes/m_tibia_frbl.stl"
+                    scale="0.01 0.01 0.01" />
+            </geometry>
+            <material name="purple" />
+        </visual>
+    </link>
+    <joint name="joint_femur_tibia_bl" type="revolute">
+        <parent link="bl_femur" />
+        <child link="bl_tibia" />
+        <origin rpy="0 0 0" xyz="0.0 -0.46 0" />
+        <axis xyz="1 0 0"/>
+        <limit lower="-${4*PI/5}" upper="0" effort="${effort}" velocity="${velocity}" />
+    </joint>
 </robot>

File: src/spiderbot_description/urdf/_front_left_leg.xacro (robot description, xacro)
@@ -35,3 +35,20 @@
         <limit lower="-${PI/4}" upper="${PI/2}" effort="${effort}" velocity="${velocity}" />
     </joint>
+    <link name="fl_tibia">
+        <visual>
+            <origin rpy="${PI} 0 0" xyz="-0.01 -0.26 0.0" />
+            <geometry>
+                <mesh filename="package://spiderbot_description/meshes/m_tibia_flbr.stl"
+                    scale="0.01 0.01 0.01" />
+            </geometry>
+            <material name="pink" />
+        </visual>
+    </link>
+    <joint name="joint_femur_tibia_fl" type="revolute">
+        <parent link="fl_femur" />
+        <child link="fl_tibia" />
+        <origin rpy="0 0 0" xyz="0.0 -0.46 0" />
+        <axis xyz="1 0 0"/>
+        <limit lower="-${4*PI/5}" upper="0" effort="${effort}" velocity="${velocity}" />
+    </joint>
 </robot>

File: src/spiderbot_description/urdf/spiderbot_colors.xacro (robot description, xacro)
@@ -25,6 +25,12 @@
     <color rgba="1.0 1.0 1.0 1.0"/>
   </material>
-    <material name="yellow">
+  <material name="yellow">
     <color rgba="1.0 1.0 0.0 1.0"/>
   </material>
+  <material name="pink">
+    <color rgba="1.0 0.75 0.79 1.0"/>
+  </material>
+  <material name="purple">
+    <color rgba="0.5 0.0 0.5 1.0"/>
+  </material>
 </robot>

Commit message: ROS2 control interface definition Collisions

File: src/spiderbot_description/urdf/_back_left_leg.xacro (robot description, xacro)
@@ -10,4 +10,12 @@
             <material name="orange" />
         </visual>
+        <collision>
+            <origin rpy="${PI} 0 0" xyz="-0.05 0 0" />
+            <geometry>
+                <mesh filename="package://spiderbot_description/meshes/m_coxa_frbl.stl"
+                    scale="0.01 0.01 0.01" />
+            </geometry>
+            <material name="orange" />
+        </collision>
     </link>
     <joint name="joint_h_bl" type="revolute">
@@ -27,4 +35,12 @@
             <material name="yellow" />
         </visual>
+        <collision>
+            <origin rpy="${PI} 0 ${PI}" xyz="0.08 -0.23 0.0" />
+            <geometry>
+                <mesh filename="package://spiderbot_description/meshes/m_femur_frbl.stl"
+                    scale="0.01 0.01 0.01" />
+            </geometry>
+            <material name="yellow" />
+        </collision>
     </link>
     <joint name="joint_hip_femur_bl" type="revolute">
@@ -44,4 +60,12 @@
             <material name="purple" />
         </visual>
+        <collision>
+            <origin rpy="${PI} 0 0" xyz="0.01 -0.26 0.0" />
+            <geometry>
+                <mesh filename="package://spiderbot_description/meshes/m_tibia_frbl.stl"
+                    scale="0.01 0.01 0.01" />
+            </geometry>
+            <material name="purple" />
+        </collision>
     </link>
     <joint name="joint_femur_tibia_bl" type="revolute">

File: src/spiderbot_description/urdf/_back_right_leg.xacro (robot description, xacro)
@@ -10,4 +10,12 @@
             <material name="blue" />
         </visual>
+        <collision>
+            <origin rpy="0 0 ${PI}" xyz="-0.05 0 0" />
+            <geometry>
+                <mesh filename="package://spiderbot_description/meshes/m_coxa_flbr.stl"
+                    scale="0.01 0.01 0.01" />
+            </geometry>
+            <material name="blue" />
+        </collision>
     </link>
     <joint name="joint_h_br" type="revolute">
@@ -27,4 +35,12 @@
             <material name="green" />
         </visual>
+        <collision>
+            <origin rpy="0 0 ${PI}" xyz="-0.08 0.23 0.0" />
+            <geometry>
+                <mesh filename="package://spiderbot_description/meshes/m_femur_flbr.stl"
+                    scale="0.01 0.01 0.01" />
+            </geometry>
+            <material name="green" />
+        </collision>
     </link>
     <joint name="joint_hip_femur_br" type="revolute">
@@ -44,4 +60,12 @@
             <material name="pink" />
         </visual>
+        <collision>
+            <origin rpy="${PI} ${PI} ${PI}" xyz="0.01 0.26 0.0" />
+            <geometry>
+                <mesh filename="package://spiderbot_description/meshes/m_tibia_flbr.stl"
+                    scale="0.01 0.01 0.01" />
+            </geometry>
+            <material name="pink" />
+        </collision>
     </link>
     <joint name="joint_femur_tibia_br" type="revolute">

File: src/spiderbot_description/urdf/_front_left_leg.xacro (robot description, xacro)
@@ -10,4 +10,12 @@
             <material name="blue" />
         </visual>
+        <collision>
+            <origin rpy="${PI} 0 ${PI}" xyz="-0.05 0 0" />
+            <geometry>
+                <mesh filename="package://spiderbot_description/meshes/m_coxa_flbr.stl"
+                    scale="0.01 0.01 0.01" />
+            </geometry>
+            <material name="blue" />
+        </collision>
     </link>
     <joint name="joint_h_fl" type="revolute">
@@ -27,4 +35,12 @@
             <material name="green" />
         </visual>
+        <collision>
+            <origin rpy="${PI} 0 ${PI}" xyz="-0.08 -0.23 0.0" />
+            <geometry>
+                <mesh filename="package://spiderbot_description/meshes/m_femur_flbr.stl"
+                    scale="0.01 0.01 0.01" />
+            </geometry>
+            <material name="green" />
+        </collision>
     </link>
     <joint name="joint_hip_femur_fl" type="revolute">
@@ -44,4 +60,12 @@
             <material name="pink" />
         </visual>
+        <collision>
+            <origin rpy="${PI} 0 0" xyz="-0.01 -0.26 0.0" />
+            <geometry>
+                <mesh filename="package://spiderbot_description/meshes/m_tibia_flbr.stl"
+                    scale="0.01 0.01 0.01" />
+            </geometry>
+            <material name="pink" />
+        </collision>
     </link>
     <joint name="joint_femur_tibia_fl" type="revolute">

File: src/spiderbot_description/urdf/_front_right_leg.xacro (robot description, xacro)
@@ -10,4 +10,12 @@
             <material name="orange" />
         </visual>
+        <collision>
+            <origin rpy="0 0 ${PI}" xyz="0.05 0 0" />
+            <geometry>
+                <mesh filename="package://spiderbot_description/meshes/m_coxa_frbl.stl"
+                    scale="0.01 0.01 0.01" />
+            </geometry>
+            <material name="orange" />
+        </collision>
     </link>
     <joint name="joint_h_fr" type="revolute">
@@ -27,4 +35,12 @@
             <material name="yellow" />
         </visual>
+        <collision>
+            <origin rpy="${PI} ${PI} 0" xyz="0.08 0.23 0.0" />
+            <geometry>
+                <mesh filename="package://spiderbot_description/meshes/m_femur_frbl.stl"
+                    scale="0.01 0.01 0.01" />
+            </geometry>
+            <material name="yellow" />
+        </collision>
     </link>
     <joint name="joint_hip_femur_fr" type="revolute">
@@ -44,4 +60,12 @@
             <material name="purple" />
         </visual>
+        <collision>
+            <origin rpy="${PI} ${PI} ${PI}" xyz="0.01 0.26 0.0" />
+            <geometry>
+                <mesh filename="package://spiderbot_description/meshes/m_tibia_frbl.stl"
+                    scale="0.01 0.01 0.01" />
+            </geometry>
+            <material name="purple" />
+        </collision>
     </link>
     <joint name="joint_femur_tibia_fr" type="revolute">

File: src/spiderbot_description/urdf/spiderbot_gazebo.xacro (robot description, xacro)
@@ -1,3 +1,26 @@
 <?xml version="1.0"?>
 <robot xmlns:xacro="http://www.ros.org/wiki/xacro">
+    <gazebo>
+        <!-- ROS 2 Humble -->
+        <xacro:if value="$(arg is_ignition)">
+            <plugin filename="ign_ros2_control-system"
+                name="ign_ros2_control::IgnitionROS2ControlPlugin">
+                <parameters>$(find arduinobot_controller)/config/arduinobot_controllers.yaml</parameters>
+            </plugin>
+            <plugin filename="ignition-gazebo-sensors-system"
+                name="ignition::gazebo::systems::Sensors">
+                <render_engine>ogre2</render_engine>
+            </plugin>
+        </xacro:if>
+        <!-- ROS 2 Iron or above -->
+        <xacro:unless value="$(arg is_ignition)">
+            <plugin filename="gz_ros2_control-system"
+                name="gz_ros2_control::GazeboSimROS2ControlPlugin">
+                <parameters>$(find arduinobot_controller)/config/arduinobot_controllers.yaml</parameters>
+            </plugin>
+            <plugin filename="gz-sim-sensors-system" name="gz::sim::systems::Sensors">
+                <render_engine>ogre2</render_engine>
+            </plugin>
+        </xacro:unless>
+    </gazebo>
 </robot>

Commit message: added inertials and gazebo launch

File: src/spiderbot_description/urdf/_back_left_leg.xacro (robot description, xacro)
@@ -2,4 +2,5 @@
 <robot xmlns:xacro="http://www.ros.org/wiki/xacro">
     <link name="bl_hip">
+        <xacro:default_inertial mass="0.02" />
         <visual>
             <origin rpy="${PI} 0 0" xyz="-0.05 0 0" />
@@ -27,4 +28,5 @@
     </joint>
     <link name="bl_femur">
+        <xacro:default_inertial mass="0.02" />
         <visual>
             <origin rpy="${PI} 0 ${PI}" xyz="0.08 -0.23 0.0" />
@@ -52,4 +54,5 @@
     </joint>
     <link name="bl_tibia">
+        <xacro:default_inertial mass="0.02" />
         <visual>
             <origin rpy="${PI} 0 0" xyz="0.01 -0.26 0.0" />

File: src/spiderbot_description/urdf/_back_right_leg.xacro (robot description, xacro)
@@ -2,4 +2,5 @@
 <robot xmlns:xacro="http://www.ros.org/wiki/xacro">
     <link name="br_hip">
+        <xacro:default_inertial mass="0.02" />
         <visual>
             <origin rpy="0 0 ${PI}" xyz="-0.05 0 0" />
@@ -27,4 +28,5 @@
     </joint>
     <link name="br_femur">
+        <xacro:default_inertial mass="0.02" />
         <visual>
             <origin rpy="0 0 ${PI}" xyz="-0.08 0.23 0.0" />
@@ -52,4 +54,5 @@
     </joint>
     <link name="br_tibia">
+        <xacro:default_inertial mass="0.02" />
         <visual>
             <origin rpy="${PI} ${PI} ${PI}" xyz="0.01 0.26 0.0" />

File: src/spiderbot_description/urdf/_front_left_leg.xacro (robot description, xacro)
@@ -2,4 +2,5 @@
 <robot xmlns:xacro="http://www.ros.org/wiki/xacro">
     <link name="fl_hip">
+        <xacro:default_inertial mass="0.02" />
         <visual>
             <origin rpy="${PI} 0 ${PI}" xyz="-0.05 0 0" />
@@ -27,4 +28,5 @@
     </joint>
     <link name="fl_femur">
+        <xacro:default_inertial mass="0.02" />
         <visual>
             <origin rpy="${PI} 0 ${PI}" xyz="-0.08 -0.23 0.0" />
@@ -52,4 +54,5 @@
     </joint>
     <link name="fl_tibia">
+        <xacro:default_inertial mass="0.02" />
         <visual>
             <origin rpy="${PI} 0 0" xyz="-0.01 -0.26 0.0" />

File: src/spiderbot_description/urdf/_front_right_leg.xacro (robot description, xacro)
@@ -2,4 +2,5 @@
 <robot xmlns:xacro="http://www.ros.org/wiki/xacro">
     <link name="fr_hip">
+        <xacro:default_inertial mass="0.02" />
         <visual>
             <origin rpy="0 0 ${PI}" xyz="0.05 0 0" />
@@ -27,4 +28,5 @@
     </joint>
     <link name="fr_femur">
+        <xacro:default_inertial mass="0.02" />
         <visual>
             <origin rpy="${PI} ${PI} 0" xyz="0.08 0.23 0.0" />
@@ -52,4 +54,5 @@
     </joint>
     <link name="fr_tibia">
+        <xacro:default_inertial mass="0.02" />
         <visual>
             <origin rpy="${PI} ${PI} ${PI}" xyz="0.01 0.26 0.0" />

File: src/spiderbot_description/urdf/spiderbot.urdf.xacro (robot description, xacro)
@@ -20,5 +20,5 @@
     <link name="base_footprint" />
     <link name="base_link">
-        <xacro:default_inertial mass="1.0" />
+        <xacro:default_inertial mass="0.110" />
         <visual>
             <origin rpy="0 0 0" xyz="0 0 0.0" />
@@ -29,4 +29,12 @@
             <material name="red" />
         </visual>
+        <collision>
+            <origin rpy="0 0 0" xyz="0 0 0.0" />
+            <geometry>
+                <mesh filename="package://spiderbot_description/meshes/m_body.stl"
+                    scale="0.01 0.01 0.01" />
+            </geometry>
+            <material name="red" />
+        </collision>
     </link>
     <joint name="base_joint" type="fixed">
