Commit message: fixed configurations issues fixed names mismatches in various places set lift, set-ready and ready group states

File: src/spiderbot_description/urdf/_back_left_leg.xacro (robot description, xacro)
@@ -21,5 +21,5 @@
     </link>
     <joint name="joint_h_bl" type="revolute">
-        <parent link="base_link" />
+        <parent link="robot_body" />
         <child link="bl_hip" />
         <origin rpy="${PI} 0 0" xyz="-0.4 -0.37 0.06" />

File: src/spiderbot_description/urdf/_back_right_leg.xacro (robot description, xacro)
@@ -21,5 +21,5 @@
     </link>
     <joint name="joint_h_br" type="revolute">
-        <parent link="base_link" />
+        <parent link="robot_body" />
         <child link="br_hip" />
         <origin rpy="0 0 ${PI}" xyz="0.4 -0.37 0.06" />

File: src/spiderbot_description/urdf/_front_left_leg.xacro (robot description, xacro)
@@ -21,5 +21,5 @@
     </link>
     <joint name="joint_h_fl" type="revolute">
-        <parent link="base_link" />
+        <parent link="robot_body" />
         <child link="fl_hip" />
         <origin rpy="${PI} 0 0" xyz="-0.4 0.37 0.06" />

File: src/spiderbot_description/urdf/_front_right_leg.xacro (robot description, xacro)
@@ -21,5 +21,5 @@
     </link>
     <joint name="joint_h_fr" type="revolute">
-        <parent link="base_link" />
+        <parent link="robot_body" />
         <child link="fr_hip" />
         <origin rpy="0 0 0" xyz="0.4 0.37 0.06" />

File: src/spiderbot_description/urdf/spiderbot.urdf.xacro (robot description, xacro)
@@ -5,6 +5,6 @@
     <xacro:arg name="is_sim" default="true" />
     <xacro:include filename="$(find spiderbot_description)/urdf/spiderbot_colors.xacro" />
-    <!-- <xacro:include filename="$(find spiderbot_description)/urdf/spiderbot_gazebo.xacro" />
-    <xacro:include filename="$(find spiderbot_description)/urdf/spiderbot_ros2_control.xacro" /> -->
+    <xacro:include filename="$(find spiderbot_description)/urdf/spiderbot_gazebo.xacro" />
+    <xacro:include filename="$(find spiderbot_description)/urdf/spiderbot_ros2_control.xacro" />
     <xacro:property name="PI" value="3.14159" />
     <xacro:property name="effort" value="30.0" />
@@ -19,5 +19,5 @@
     </xacro:macro>
     <link name="base_footprint" />
-    <link name="base_link">
+    <link name="robot_body">
         <xacro:default_inertial mass="0.110" />
         <visual>
@@ -38,7 +38,7 @@
         </collision>
     </link>
-    <joint name="base_joint" type="fixed">
+    <joint name="virtual_joint" type="fixed">
         <parent link="base_footprint" />
-        <child link="base_link" />
+        <child link="robot_body" />
         <origin rpy="0 0 0" xyz="0 0 0.3" />
     </joint>

File: src/spiderbot_description/urdf/spiderbot_gazebo.xacro (robot description, xacro)
@@ -6,5 +6,5 @@
             <plugin filename="ign_ros2_control-system"
                 name="ign_ros2_control::IgnitionROS2ControlPlugin">
-                <parameters>$(find arduinobot_controller)/config/arduinobot_controllers.yaml</parameters>
+                <parameters>$(find spiderbot_controllers)/config/spiderbot_controllers.yaml</parameters>
             </plugin>
             <plugin filename="ignition-gazebo-sensors-system"
@@ -17,5 +17,5 @@
             <plugin filename="gz_ros2_control-system"
                 name="gz_ros2_control::GazeboSimROS2ControlPlugin">
-                <parameters>$(find arduinobot_controller)/config/arduinobot_controllers.yaml</parameters>
+                <parameters>$(find spiderbot_controllers)/config/spiderbot_controllers.yaml</parameters>
             </plugin>
             <plugin filename="gz-sim-sensors-system" name="gz::sim::systems::Sensors">

Commit message: Recolored the model more logically

File: src/spiderbot_description/urdf/_back_left_leg.xacro (robot description, xacro)
@@ -9,5 +9,5 @@
                     scale="0.01 0.01 0.01" />
             </geometry>
-            <material name="orange" />
+            <material name="blue" />
         </visual>
         <collision>
@@ -17,5 +17,4 @@
                     scale="0.01 0.01 0.01" />
             </geometry>
-            <material name="orange" />
         </collision>
     </link>
@@ -43,5 +42,4 @@
                     scale="0.01 0.01 0.01" />
             </geometry>
-            <material name="yellow" />
         </collision>
     </link>
@@ -61,5 +59,5 @@
                     scale="0.01 0.01 0.01" />
             </geometry>
-            <material name="purple" />
+            <material name="red" />
         </visual>
         <collision>
@@ -69,5 +67,4 @@
                     scale="0.01 0.01 0.01" />
             </geometry>
-            <material name="purple" />
         </collision>
     </link>

File: src/spiderbot_description/urdf/_back_right_leg.xacro (robot description, xacro)
@@ -17,5 +17,4 @@
                     scale="0.01 0.01 0.01" />
             </geometry>
-            <material name="blue" />
         </collision>
     </link>
@@ -35,5 +34,5 @@
                     scale="0.01 0.01 0.01" />
             </geometry>
-            <material name="green" />
+            <material name="yellow" />
         </visual>
         <collision>
@@ -43,5 +42,4 @@
                     scale="0.01 0.01 0.01" />
             </geometry>
-            <material name="green" />
         </collision>
     </link>
@@ -61,5 +59,5 @@
                     scale="0.01 0.01 0.01" />
             </geometry>
-            <material name="pink" />
+            <material name="green" />
         </visual>
         <collision>
@@ -69,5 +67,4 @@
                     scale="0.01 0.01 0.01" />
             </geometry>
-            <material name="pink" />
         </collision>
     </link>

File: src/spiderbot_description/urdf/_front_left_leg.xacro (robot description, xacro)
@@ -17,5 +17,4 @@
                     scale="0.01 0.01 0.01" />
             </geometry>
-            <material name="blue" />
         </collision>
     </link>
@@ -35,5 +34,5 @@
                     scale="0.01 0.01 0.01" />
             </geometry>
-            <material name="green" />
+            <material name="yellow" />
         </visual>
         <collision>
@@ -43,5 +42,4 @@
                     scale="0.01 0.01 0.01" />
             </geometry>
-            <material name="green" />
         </collision>
     </link>
@@ -61,5 +59,5 @@
                     scale="0.01 0.01 0.01" />
             </geometry>
-            <material name="pink" />
+            <material name="red" />
         </visual>
         <collision>
@@ -69,5 +67,4 @@
                     scale="0.01 0.01 0.01" />
             </geometry>
-            <material name="pink" />
         </collision>
     </link>

File: src/spiderbot_description/urdf/_front_right_leg.xacro (robot description, xacro)
@@ -9,5 +9,5 @@
                     scale="0.01 0.01 0.01" />
             </geometry>
-            <material name="orange" />
+            <material name="blue" />
         </visual>
         <collision>
@@ -17,5 +17,4 @@
                     scale="0.01 0.01 0.01" />
             </geometry>
-            <material name="orange" />
         </collision>
     </link>
@@ -43,5 +42,4 @@
                     scale="0.01 0.01 0.01" />
             </geometry>
-            <material name="yellow" />
         </collision>
     </link>
@@ -61,5 +59,5 @@
                     scale="0.01 0.01 0.01" />
             </geometry>
-            <material name="purple" />
+            <material name="green" />
         </visual>
         <collision>
@@ -69,5 +67,4 @@
                     scale="0.01 0.01 0.01" />
             </geometry>
-            <material name="purple" />
         </collision>
     </link>

File: src/spiderbot_description/urdf/spiderbot.urdf.xacro (robot description, xacro)
@@ -27,5 +27,5 @@
                     scale="0.01 0.01 0.01" />
             </geometry>
-            <material name="red" />
+            <material name="purple" />
         </visual>
         <collision>
@@ -35,5 +35,4 @@
                     scale="0.01 0.01 0.01" />
             </geometry>
-            <material name="red" />
         </collision>
     </link>

File: src/spiderbot_description/urdf/spiderbot_colors.xacro (robot description, xacro)
@@ -14,5 +14,5 @@
   </material>
   <material name="orange">
-    <color rgba="${255/255} ${108/255} ${10/255} 1.0"/>
+    <color rgba="${255/255} ${102/255} 0 1.0"/>
   </material>
   <material name="brown">
